Commit message: Removed XACRO because not compatible with Eloquent

File: zed_wrapper/urdf/zed.urdf (robot description, URDF)
Before this commit: robot zed_camera, 6 links, 5 joints
Links:
- link zed_camera_center: geometry visual mesh filename=package://stereolabs_zed/urdf/models/zed.stl

File: zed_wrapper/urdf/zed2.urdf (robot description, URDF)
Before this commit: robot zedm_camera, 6 links, 5 joints
Links:
- removed link zed_camera_center
- removed link zed_left_camera_frame
- removed link zed_left_camera_optical_frame
- removed link zed_right_camera_frame
- removed link zed_right_camera_optical_frame
- added link zed2_camera_center; visual mesh filename=package://stereolabs_zed/urdf/models/zed2.stl
- added link zed2_left_camera_frame
- added link zed2_left_camera_optical_frame
- added link zed2_right_camera_frame
- added link zed2_right_camera_optical_frame
Joints:
- removed joint zed_camera_center_joint
- removed joint zed_left_camera_joint
- removed joint zed_left_camera_optical_joint
- removed joint zed_right_camera_joint
- removed joint zed_right_camera_optical_joint
- added joint zed2_camera_center_joint: type fixed, parent base_link, child zed2_camera_center, origin xyz=0 0 0 rpy=0 0 0
- added joint zed2_left_camera_joint: type fixed, parent zed2_camera_center, child zed2_left_camera_frame, origin xyz=0 0.06 0 rpy=0 0 0
- added joint zed2_left_camera_optical_joint: type fixed, parent zed2_left_camera_frame, child zed2_left_camera_optical_frame, origin xyz=0 0 0 rpy=-1.57079632679 0.0 -1.57079632679
- added joint zed2_right_camera_joint: type fixed, parent zed2_camera_center, child zed2_right_camera_frame, origin xyz=0 -0.06 0 rpy=0 0 0
- added joint zed2_right_camera_optical_joint: type fixed, parent zed2_right_camera_frame, child zed2_right_camera_optical_frame, origin xyz=0 0 0 rpy=-1.57079632679 0.0 -1.57079632679

File: zed_wrapper/urdf/zedm.urdf (robot description, URDF)
Before this commit: robot zedm_camera, 6 links, 5 joints
Links:
- removed link zed_camera_center
- removed link zed_left_camera_frame
- removed link zed_left_camera_optical_frame
- removed link zed_right_camera_frame
- removed link zed_right_camera_optical_frame
- added link zedm_camera_center; visual mesh filename=package://stereolabs_zed/urdf/models/zedm.stl
- added link zedm_left_camera_frame
- added link zedm_left_camera_optical_frame
- added link zedm_right_camera_frame
- added link zedm_right_camera_optical_frame
Joints:
- removed joint zed_camera_center_joint
- removed joint zed_left_camera_joint
- removed joint zed_left_camera_optical_joint
- removed joint zed_right_camera_joint
- removed joint zed_right_camera_optical_joint
- added joint zedm_camera_center_joint: type fixed, parent base_link, child zedm_camera_center, origin xyz=0 0 0 rpy=0 0 0
- added joint zedm_left_camera_joint: type fixed, parent zedm_camera_center, child zedm_left_camera_frame, origin xyz=0 0.03 0 rpy=0 0 0
- added joint zedm_left_camera_optical_joint: type fixed, parent zedm_left_camera_frame, child zedm_left_camera_optical_frame, origin xyz=0 0 0 rpy=-1.57079632679 0.0 -1.57079632679
- added joint zedm_right_camera_joint: type fixed, parent zedm_camera_center, child zedm_right_camera_frame, origin xyz=0 -0.03 0 rpy=0 0 0
- added joint zedm_right_camera_optical_joint: type fixed, parent zedm_right_camera_frame, child zedm_right_camera_optical_frame, origin xyz=0 0 0 rpy=-1.57079632679 0.0 -1.57079632679

Commit message: Fix camera_info topic issue

File: zed_wrapper/urdf/zed.urdf (robot description, URDF)
Before this commit: robot zed_camera, 6 links, 5 joints
Links:
- link zed_camera_center: geometry visual mesh filename=package://zed_wrapper/urdf/models/zed.stl

File: zed_wrapper/urdf/zed2.urdf (robot description, URDF)
Before this commit: robot zed2_camera, 6 links, 5 joints
Links:
- link zed2_camera_center: geometry visual mesh filename=package://zed_wrapper/urdf/models/zed2.stl

File: zed_wrapper/urdf/zedm.urdf (robot description, URDF)
Before this commit: robot zedm_camera, 6 links, 5 joints
Links:
- link zedm_camera_center: geometry visual mesh filename=package://zed_wrapper/urdf/models/zedm.stl
