Commit message: Cleanup

File: zed_wrapper/urdf/zed2.urdf (robot description, URDF)
Before this commit: robot zed2_camera, 6 links, 5 joints
Links:
- removed link base_link
- added link zed_link
Joints:
- joint zed2_camera_center_joint: parent base_link -> zed_link

Commit message: Prepare PR

File: zed_wrapper/urdf/zed2.urdf (robot description, URDF)
Before this commit: robot zed2_camera, 6 links, 5 joints
Links:
- removed link zed_link
- added link base_link
Joints:
- joint zed2_camera_center_joint: parent zed_link -> base_link
