Commit message: Remove zed_interfaces files and add the submodule

File: zed_wrapper/urdf/zed_macro.urdf.xacro (robot description, xacro)
@@ -66,5 +66,5 @@
         <origin xyz="${screw_offset_x} 0 0" rpy="0 0 0"/>
         <geometry>
-          <mesh filename="package://zed_wrapper/urdf/models/${model}.stl" />
+          <mesh filename="package://zed_interfaces/meshes/${model}.stl" />
         </geometry>
         <material name="${model}_mat" />
@@ -72,5 +72,5 @@
       <collision>
         <geometry>
-          <mesh filename="package://zed_wrapper/urdf/models/${model}.stl" />
+          <mesh filename="package://zed_interfaces/meshes/${model}.stl" />
         </geometry>
       </collision>

Commit message: Add support for ZED-X and ZED-X Mini

File: zed_wrapper/urdf/zed_macro.urdf.xacro (robot description, xacro)
@@ -31,4 +31,5 @@
       <xacro:property name="bottom_slope" value="0.05" />
       <xacro:property name="screw_offset_x" value="0.0" />
+      <xacro:property name="screw_offset_z" value="0.0" />
       <xacro:property name="optical_offset_x" value="-0.01" />
     </xacro:if>
@@ -38,4 +39,5 @@
       <xacro:property name="bottom_slope" value="0.0" />
       <xacro:property name="screw_offset_x" value="0.0" />
+      <xacro:property name="screw_offset_z" value="0.0" />
       <xacro:property name="optical_offset_x" value="0.0" />
     </xacro:if>
@@ -45,4 +47,5 @@
       <xacro:property name="bottom_slope" value="0.05" />
       <xacro:property name="screw_offset_x" value="0.0" />
+      <xacro:property name="screw_offset_z" value="0.0" />
       <xacro:property name="optical_offset_x" value="-0.01" />
     </xacro:if>
@@ -52,4 +55,21 @@
       <xacro:property name="bottom_slope" value="0.0" />
       <xacro:property name="screw_offset_x" value="-0.01" />
+      <xacro:property name="screw_offset_z" value="0.0" />
+      <xacro:property name="optical_offset_x" value="-0.01" />
+    </xacro:if>
+    <xacro:if value="${model == 'zedx'}">
+      <xacro:property name="baseline" value="0.12" />
+      <xacro:property name="height" value="0.032" />
+      <xacro:property name="bottom_slope" value="0.0" />
+      <xacro:property name="screw_offset_x" value="0.0" />
+      <xacro:property name="screw_offset_z" value="-0.016" />
+      <xacro:property name="optical_offset_x" value="-0.01" />
+    </xacro:if>
+    <xacro:if value="${model == 'zedxm'}">
+      <xacro:property name="baseline" value="0.05" />
+      <xacro:property name="height" value="0.032" />
+      <xacro:property name="bottom_slope" value="0.0" />
+      <xacro:property name="screw_offset_x" value="0.0" />
+      <xacro:property name="screw_offset_z" value="-0.016" />
       <xacro:property name="optical_offset_x" value="-0.01" />
     </xacro:if>
@@ -64,5 +84,5 @@
     <link name="${name}_camera_center">
       <visual>
-        <origin xyz="${screw_offset_x} 0 0" rpy="0 0 0"/>
+        <origin xyz="${screw_offset_x} 0 ${screw_offset_z}" rpy="0 0 0"/>
         <geometry>
           <mesh filename="package://zed_interfaces/meshes/${model}.stl" />
@@ -86,9 +106,9 @@
       <parent link="${name}_camera_center"/>
       <child link="${name}_left_camera_frame"/>
-      <origin xyz="0 ${baseline/2} 0" rpy="0 0 0" />
+      <origin xyz="${optical_offset_x} ${baseline/2} 0" rpy="0 0 0" />
     </joint>
     <link name="${name}_left_camera_optical_frame"/>
     <joint name="${name}_left_camera_optical_joint" type="fixed">
-      <origin xyz="${optical_offset_x} 0 0" rpy="-${M_PI/2} 0.0 -${M_PI/2}"/>
+      <origin xyz="0 0 0" rpy="-${M_PI/2} 0.0 -${M_PI/2}"/>
       <parent link="${name}_left_camera_frame"/>
       <child link="${name}_left_camera_optical_frame"/>
@@ -99,9 +119,9 @@
       <parent link="${name}_camera_center"/>
       <child link="${name}_right_camera_frame"/>
-      <origin xyz="0 -${baseline/2} 0" rpy="0 0 0" />
+      <origin xyz="${optical_offset_x} -${baseline/2} 0" rpy="0 0 0" />
     </joint>
     <link name="${name}_right_camera_optical_frame"/>
     <joint name="${name}_right_camera_optical_joint" type="fixed">
-      <origin xyz="${optical_offset_x} 0 0" rpy="-${M_PI/2} 0.0 -${M_PI/2}"/>
+      <origin xyz="0 0 0" rpy="-${M_PI/2} 0.0 -${M_PI/2}"/>
       <parent link="${name}_right_camera_frame"/>
       <child link="${name}_right_camera_optical_frame"/>

Commit message: Fix xacro offset

File: zed_wrapper/urdf/zed_macro.urdf.xacro (robot description, xacro)
@@ -84,4 +84,5 @@
       </visual>
       <collision>
+        <origin xyz="${screw_offset_x} 0 ${screw_offset_z}" rpy="0 0 0"/>
         <geometry>
           <mesh filename="package://zed_interfaces/meshes/${model}.stl" />

Commit message: Update zed_macro.urdf.xacro

File: zed_wrapper/urdf/zed_macro.urdf.xacro (robot description, xacro)
@@ -17,5 +17,8 @@
 <robot xmlns:xacro="http://wiki.ros.org/xacro">
   <xacro:include filename="$(find zed_wrapper)/urdf/include/materials.urdf.xacro" />
-  <xacro:property name="M_PI"     value="3.1415926535897931" />
+  <xacro:property name="M_PI"       value="3.1415926535897931" />
+  <xacro:property name="cam_depth"  value="0.037298" />
+  <xacro:property name="cam_width"  value="0.17525" />
+  <xacro:property name="cam_height" value="0.03025" />
   <!--
     Parameters:
@@ -79,12 +82,12 @@
         <origin xyz="${screw_offset_x} 0 ${screw_offset_z}" rpy="0 0 0"/>
         <geometry>
-          <mesh filename="package://zed_interfaces/meshes/${model}.stl" />
+          <box size="${cam_depth} ${cam_width} ${cam_height}"/>
         </geometry>
-        <material name="${model}_mat" />
+        <material name="white"/>
       </visual>
       <collision>
         <origin xyz="${screw_offset_x} 0 ${screw_offset_z}" rpy="0 0 0"/>
         <geometry>
-          <mesh filename="package://zed_interfaces/meshes/${model}.stl" />
+          <box size="${cam_depth} ${cam_width} ${cam_height}"/>
         </geometry>
       </collision>

Commit message: Changed the name of the package `zed_interfaces` to `zed_msgs` to match the ROS2 naming convention

File: zed_wrapper/urdf/zed_macro.urdf.xacro (robot description, xacro)
@@ -89,5 +89,5 @@
           <origin xyz="${screw_offset_x} 0 ${screw_offset_z}" rpy="0 0 0"/>
           <geometry>
-            <mesh filename="package://zed_interfaces/meshes/${model}.stl" />
+<mesh filename="package://zed_msgs/meshes/${model}.stl" />
           </geometry>
           <material name="${model}_mat" />
@@ -96,5 +96,5 @@
           <origin xyz="${screw_offset_x} 0 ${screw_offset_z}" rpy="0 0 0"/>
           <geometry>
-            <mesh filename="package://zed_interfaces/meshes/${model}.stl" />
+<mesh filename="package://zed_msgs/meshes/${model}.stl" />
           </geometry>
         </collision>
@@ -112,5 +112,5 @@
           <origin xyz="0 0 0" rpy="0 0 0"/>
           <geometry>
-            <mesh filename="package://zed_interfaces/meshes/${model}.stl" />
+<mesh filename="package://zed_msgs/meshes/${model}.stl" />
           </geometry>
           <material name="${model}_mat" />
@@ -119,5 +119,5 @@
           <origin xyz="0 0 0" rpy="0 0 0"/>
           <geometry>
-            <mesh filename="package://zed_interfaces/meshes/${model}.stl" />
+<mesh filename="package://zed_msgs/meshes/${model}.stl" />
           </geometry>
         </collision>
@@ -141,5 +141,5 @@
           <origin xyz="0 0 0" rpy="0 0 0"/>
           <geometry>
-            <mesh filename="package://zed_interfaces/meshes/${model}.stl" />
+<mesh filename="package://zed_msgs/meshes/${model}.stl" />
           </geometry>
           <material name="${model}_mat" />
@@ -148,5 +148,5 @@
           <origin xyz="0 0 0" rpy="0 0 0"/>
           <geometry>
-            <mesh filename="package://zed_interfaces/meshes/${model}.stl" />
+<mesh filename="package://zed_msgs/meshes/${model}.stl" />
           </geometry>
         </collision>

Commit message: Change ZEDM distance according to the datasheet

File: zed_wrapper/urdf/zed_macro.urdf.xacro (robot description, xacro)
@@ -35,5 +35,5 @@
     </xacro:if>
     <xacro:if value="${model == 'zedm'}">
-      <xacro:property name="baseline" value="0.06" />
+      <xacro:property name="baseline" value="0.063" />
       <xacro:property name="height" value="0.0265" />
       <xacro:property name="bottom_slope" value="0.0" />

Commit message: Updated fix works with both RVIZ2 and Gazebo

File: zed_wrapper/urdf/zed_macro.urdf.xacro (robot description, xacro)
@@ -114,5 +114,5 @@
           <origin xyz="${screw_offset_x} 0 ${screw_offset_z}" rpy="0 0 0"/>
           <geometry>
-<mesh filename="$(find zed_msgs)/meshes/${model}.stl" />
+<mesh filename="file://$(find zed_msgs)/meshes/${model}.stl"/>
           </geometry>
           <material name="${model}_mat" />
@@ -121,5 +121,5 @@
           <origin xyz="${screw_offset_x} 0 ${screw_offset_z}" rpy="0 0 0"/>
           <geometry>
-<mesh filename="$(find zed_msgs)/meshes/${model}.stl" />
+<mesh filename="file://$(find zed_msgs)/meshes/${model}.stl"/>
           </geometry>
         </collision>
@@ -138,5 +138,5 @@
             <origin xyz="0 0 0" rpy="0 0 0"/>
             <geometry>
-  <mesh filename="$(find zed_msgs)/meshes/${model}.stl" />
+  <mesh filename="file://$(find zed_msgs)/meshes/${model}.stl"/>
             </geometry>
             <material name="${model}_mat" />
@@ -145,5 +145,5 @@
             <origin xyz="0 0 0" rpy="0 0 0"/>
             <geometry>
-  <mesh filename="$(find zed_msgs)/meshes/${model}.stl" />
+  <mesh filename="file://$(find zed_msgs)/meshes/${model}.stl"/>
             </geometry>
           </collision>
@@ -167,5 +167,5 @@
             <origin xyz="0 0 0" rpy="0 0 0"/>
             <geometry>
-  <mesh filename="$(find zed_msgs)/meshes/${model}.stl" />
+  <mesh filename="file://$(find zed_msgs)/meshes/${model}.stl"/>
             </geometry>
             <material name="${model}_mat" />
@@ -174,5 +174,5 @@
             <origin xyz="0 0 0" rpy="0 0 0"/>
             <geometry>
-  <mesh filename="$(find zed_msgs)/meshes/${model}.stl" />
+  <mesh filename="file://$(find zed_msgs)/meshes/${model}.stl"/>
             </geometry>
           </collision>

Commit message: Minor fix

File: zed_wrapper/urdf/zed_macro.urdf.xacro (robot description, xacro)
@@ -150,5 +150,5 @@
           <origin xyz="${screw_offset_x} 0 ${screw_offset_z}" rpy="0 0 0"/>
           <geometry>
-<mesh filename="file://$(find zed_msgs)/meshes/${model}.stl"/>
+            <mesh filename="file://$(find zed_msgs)/meshes/${model}.stl"/>
           </geometry>
           <material name="${model}_mat" />
@@ -157,5 +157,5 @@
           <origin xyz="${screw_offset_x} 0 ${screw_offset_z}" rpy="0 0 0"/>
           <geometry>
-<mesh filename="file://$(find zed_msgs)/meshes/${model}.stl"/>
+            <mesh filename="file://$(find zed_msgs)/meshes/${model}.stl"/>
           </geometry>
         </collision>
@@ -174,5 +174,5 @@
             <origin xyz="0 0 0" rpy="0 0 0"/>
             <geometry>
-  <mesh filename="file://$(find zed_msgs)/meshes/${model}.stl"/>
+              <mesh filename="file://$(find zed_msgs)/meshes/${model}.stl"/>
             </geometry>
             <material name="${model}_mat" />
@@ -181,5 +181,5 @@
             <origin xyz="0 0 0" rpy="0 0 0"/>
             <geometry>
-  <mesh filename="file://$(find zed_msgs)/meshes/${model}.stl"/>
+              <mesh filename="file://$(find zed_msgs)/meshes/${model}.stl"/>
             </geometry>
           </collision>
@@ -203,5 +203,5 @@
             <origin xyz="0 0 0" rpy="0 0 0"/>
             <geometry>
-  <mesh filename="file://$(find zed_msgs)/meshes/${model}.stl"/>
+              <mesh filename="file://$(find zed_msgs)/meshes/${model}.stl"/>
             </geometry>
             <material name="${model}_mat" />
@@ -210,5 +210,5 @@
             <origin xyz="0 0 0" rpy="0 0 0"/>
             <geometry>
-  <mesh filename="file://$(find zed_msgs)/meshes/${model}.stl"/>
+              <mesh filename="file://$(find zed_msgs)/meshes/${model}.stl"/>
             </geometry>
           </collision>

Commit message: fix: update frame names to match ROS REP 103
Signed-off-by: Beniamino Pozzan <b.pozzan@archangelautonomy.com>

File: zed_wrapper/urdf/zed_macro.urdf.xacro (robot description, xacro)
@@ -191,9 +191,9 @@
         <origin xyz="${optical_offset_x} ${baseline/2} 0" rpy="0 0 0" />
       </joint>
-      <link name="${name}_left_camera_optical_frame"/>
+      <link name="${name}_left_camera_frame_optical"/>
       <joint name="${name}_left_camera_optical_joint" type="fixed">
         <origin xyz="0 0 0" rpy="-${M_PI/2} 0.0 -${M_PI/2}"/>
         <parent link="${name}_left_camera_frame"/>
-        <child link="${name}_left_camera_optical_frame"/>
+        <child link="${name}_left_camera_frame_optical"/>
       </joint>
       <!-- Right Camera -->
@@ -220,9 +220,9 @@
         <origin xyz="${optical_offset_x} -${baseline/2} 0" rpy="0 0 0" />
       </joint>
-      <link name="${name}_right_camera_optical_frame"/>
+      <link name="${name}_right_camera_frame_optical"/>
       <joint name="${name}_right_camera_optical_joint" type="fixed">
         <origin xyz="0 0 0" rpy="-${M_PI/2} 0.0 -${M_PI/2}"/>
         <parent link="${name}_right_camera_frame"/>
-        <child link="${name}_right_camera_optical_frame"/>
+        <child link="${name}_right_camera_frame_optical"/>
       </joint>
       <!-- ZED2 Sensors -->
@@ -262,9 +262,9 @@
         <origin xyz="${optical_offset_x} 0 0" rpy="0 0 0" />
       </joint>
-      <link name="${name}_camera_optical_frame"/>
+      <link name="${name}_camera_frame_optical"/>
       <joint name="${name}_camera_optical_joint" type="fixed">
         <origin xyz="0 0 0" rpy="-${M_PI/2} 0.0 -${M_PI/2}"/>
         <parent link="${name}_camera_frame"/>
-        <child link="${name}_camera_optical_frame"/>
+        <child link="${name}_camera_frame_optical"/>
       </joint>
     </xacro:if>

Commit message: Moved materials into macro

File: zed_wrapper/urdf/zed_macro.urdf.xacro (robot description, xacro)
@@ -16,5 +16,5 @@
 -->
 <robot xmlns:xacro="http://wiki.ros.org/xacro">
-  <xacro:include filename="$(find zed_wrapper)/urdf/include/materials.urdf.xacro" />
+  <!-- xacro:include filename="$(find zed_wrapper)/urdf/include/materials.urdf.xacro" / -->
   <xacro:property name="M_PI"     value="3.1415926535897931" />
   <!--
@@ -33,4 +33,5 @@
       <xacro:property name="optical_offset_x" value="-0.01" />
       <xacro:property name="mono" value="false" />
+      <xacro:property name="mat" value="0.8 0.8 0.8 1.0" />
     </xacro:if>
     <xacro:if value="${model == 'zedm'}">
@@ -42,4 +43,5 @@
       <xacro:property name="optical_offset_x" value="0.0" />
       <xacro:property name="mono" value="false" />
+      <xacro:property name="mat" value="0 0 0 1.0" />
     </xacro:if>
     <xacro:if value="${model == 'zed2'}">
@@ -51,4 +53,5 @@
       <xacro:property name="optical_offset_x" value="-0.01" />
       <xacro:property name="mono" value="false" />
+      <xacro:property name="mat" value="0.25 0.25 0.25 1.0" />
     </xacro:if>
     <xacro:if value="${model == 'zed2i'}">
@@ -60,4 +63,5 @@
       <xacro:property name="optical_offset_x" value="-0.01" />
       <xacro:property name="mono" value="false" />
+      <xacro:property name="mat" value="0.25 0.25 0.25 1.0" />
     </xacro:if>
     <xacro:if value="${model == 'zedx'}">
@@ -69,4 +73,5 @@
       <xacro:property name="optical_offset_x" value="-0.01" />
       <xacro:property name="mono" value="false" />
+      <xacro:property name="mat" value="0.25 0.25 0.25 1.0" />
     </xacro:if>
     <xacro:if value="${model == 'zedxhdr'}">
@@ -78,4 +83,5 @@
       <xacro:property name="optical_offset_x" value="-0.01" />
       <xacro:property name="mono" value="false" />
+      <xacro:property name="mat" value="0.25 0.25 0.25 1.0" />
     </xacro:if>
     <xacro:if value="${model == 'zedxm'}">
@@ -87,4 +93,5 @@
       <xacro:property name="optical_offset_x" value="-0.01" />
       <xacro:property name="mono" value="false" />
+      <xacro:property name="mat" value="0.25 0.25 0.25 1.0" />
     </xacro:if>
     <xacro:if value="${model == 'zedxhdrmini'}">
@@ -96,4 +103,5 @@
       <xacro:property name="optical_offset_x" value="-0.01" />
       <xacro:property name="mono" value="false" />
+      <xacro:property name="mat" value="0.25 0.25 0.25 1.0" />
     </xacro:if>
     <xacro:if value="${model == 'zedxhdrmax'}">
@@ -105,4 +113,5 @@
       <xacro:property name="optical_offset_x" value="-0.01" />
       <xacro:property name="mono" value="false" />
+      <xacro:property name="mat" value="0.25 0.25 0.25 1.0" />
     </xacro:if>
     <xacro:if value="${model == 'virtual'}">
@@ -114,4 +123,5 @@
       <xacro:property name="optical_offset_x" value="0.0" />
       <xacro:property name="mono" value="false" />
+      <xacro:property name="mat" value="0.25 0.25 0.25 1.0" />
     </xacro:if>
     <xacro:if value="${model == 'zedxonegs'}">
@@ -123,4 +133,5 @@
       <xacro:property name="optical_offset_x" value="0.0" />
       <xacro:property name="mono" value="true" />
+      <xacro:property name="mat" value="0.25 0.25 0.25 1.0" />
     </xacro:if>
     <xacro:if value="${model == 'zedxone4k'}">
@@ -132,4 +143,5 @@
       <xacro:property name="optical_offset_x" value="0.0" />
       <xacro:property name="mono" value="true" />
+      <xacro:property name="mat" value="0.25 0.25 0.25 1.0" />
     </xacro:if>
     <xacro:if value="${model == 'zedxonehdr'}">
@@ -141,4 +153,5 @@
       <xacro:property name="optical_offset_x" value="0.0" />
       <xacro:property name="mono" value="true" />
+      <xacro:property name="mat" value="0.25 0.25 0.25 1.0" />
     </xacro:if>
     <!-- Camera mounting point (the threaded screw hole in the bottom) -->
@@ -152,5 +165,7 @@
             <mesh filename="file://$(find zed_msgs)/meshes/${model}.stl"/>
           </geometry>
-          <material name="${model}_mat" />
+            <material name="zed_mat">
+              <color rgba="${mat}"/>
+            </material>
         </visual>
         <collision>
@@ -176,5 +191,7 @@
               <mesh filename="file://$(find zed_msgs)/meshes/${model}.stl"/>
             </geometry>
-            <material name="${model}_mat" />
+            <material name="zed_mat">
+              <color rgba="${mat}"/>
+            </material>
           </visual>
           <collision>
@@ -205,5 +222,7 @@
               <mesh filename="file://$(find zed_msgs)/meshes/${model}.stl"/>
             </geometry>
-            <material name="${model}_mat" />
+            <material name="zed_mat">
+              <color rgba="${mat}"/>
+            </material>
           </visual>
           <collision>
