Commit message: edit path to meshes

File: zed_wrapper/urdf/zed_macro.urdf.xacro (robot description, xacro)
@@ -172,5 +172,5 @@
           <origin xyz="${screw_offset_x} 0 ${screw_offset_z}" rpy="0 0 0"/>
           <geometry>
-            <mesh filename="file://$(find zed_msgs)/meshes/${model}.stl"/>
+            <mesh filename="file://$(find zed_description)/meshes/${model}.stl"/>
           </geometry>
             <material name="zed_mat">
@@ -181,5 +181,5 @@
           <origin xyz="${screw_offset_x} 0 ${screw_offset_z}" rpy="0 0 0"/>
           <geometry>
-            <mesh filename="file://$(find zed_msgs)/meshes/${model}.stl"/>
+            <mesh filename="file://$(find zed_description)/meshes/${model}.stl"/>
           </geometry>
         </collision>
@@ -198,5 +198,5 @@
             <origin xyz="0 0 0" rpy="0 0 0"/>
             <geometry>
-              <mesh filename="file://$(find zed_msgs)/meshes/${model}.stl"/>
+              <mesh filename="file://$(find zed_description)/meshes/${model}.stl"/>
             </geometry>
             <material name="zed_mat">
@@ -207,5 +207,5 @@
             <origin xyz="0 0 0" rpy="0 0 0"/>
             <geometry>
-              <mesh filename="file://$(find zed_msgs)/meshes/${model}.stl"/>
+              <mesh filename="file://$(find zed_description)/meshes/${model}.stl"/>
             </geometry>
           </collision>
@@ -229,5 +229,5 @@
             <origin xyz="0 0 0" rpy="0 0 0"/>
             <geometry>
-              <mesh filename="file://$(find zed_msgs)/meshes/${model}.stl"/>
+              <mesh filename="file://$(find zed_description)/meshes/${model}.stl"/>
             </geometry>
             <material name="zed_mat">
@@ -238,5 +238,5 @@
             <origin xyz="0 0 0" rpy="0 0 0"/>
             <geometry>
-              <mesh filename="file://$(find zed_msgs)/meshes/${model}.stl"/>
+              <mesh filename="file://$(find zed_description)/meshes/${model}.stl"/>
             </geometry>
           </collision>
