Commit message: Add `sl::Fusion` module for GNSS

File: zed_wrapper/urdf/include/materials.urdf.xacro (robot description, xacro)
@@ -28,3 +28,9 @@
         <color rgba="0.25 0.25 0.25 0.99"/>
     </material>
+    <material name="zedx_mat">
+        <color rgba="0.25 0.25 0.25 0.99"/>
+    </material>
+    <material name="zedxm_mat">
+        <color rgba="0.25 0.25 0.25 0.99"/>
+    </material>
 </robot>

Commit message: Add ZED X One to xacro

File: zed_wrapper/urdf/include/materials.urdf.xacro (robot description, xacro)
@@ -37,3 +37,9 @@
         <color rgba="0.25 0.25 0.25 1.0"/>
     </material>
+    <material name="zedxonegs_mat">
+        <color rgba="0.25 0.25 0.25 1.0"/>
+    </material>
+    <material name="zedxone4k_mat">
+        <color rgba="0.25 0.25 0.25 1.0"/>
+    </material>
 </robot>

File: zed_wrapper/urdf/zed_macro.urdf.xacro (robot description, xacro)
@@ -32,4 +32,5 @@
       <xacro:property name="screw_offset_z" value="0.0" />
       <xacro:property name="optical_offset_x" value="-0.01" />
+      <xacro:property name="mono" value="false" />
     </xacro:if>
     <xacro:if value="${model == 'zedm'}">
@@ -40,4 +41,5 @@
       <xacro:property name="screw_offset_z" value="0.0" />
       <xacro:property name="optical_offset_x" value="0.0" />
+      <xacro:property name="mono" value="false" />
     </xacro:if>
     <xacro:if value="${model == 'zed2'}">
@@ -48,4 +50,5 @@
       <xacro:property name="screw_offset_z" value="0.0" />
       <xacro:property name="optical_offset_x" value="-0.01" />
+      <xacro:property name="mono" value="false" />
     </xacro:if>
     <xacro:if value="${model == 'zed2i'}">
@@ -56,4 +59,5 @@
       <xacro:property name="screw_offset_z" value="0.0" />
       <xacro:property name="optical_offset_x" value="-0.01" />
+      <xacro:property name="mono" value="false" />
     </xacro:if>
     <xacro:if value="${model == 'zedx'}">
@@ -64,4 +68,5 @@
       <xacro:property name="screw_offset_z" value="-0.016" />
       <xacro:property name="optical_offset_x" value="-0.01" />
+      <xacro:property name="mono" value="false" />
     </xacro:if>
     <xacro:if value="${model == 'zedxm'}">
@@ -72,4 +77,5 @@
       <xacro:property name="screw_offset_z" value="-0.016" />
       <xacro:property name="optical_offset_x" value="-0.01" />
+      <xacro:property name="mono" value="false" />
     </xacro:if>
     <xacro:if value="${model == 'virtual'}">
@@ -80,4 +86,23 @@
       <xacro:property name="screw_offset_z" value="-0.0155" />
       <xacro:property name="optical_offset_x" value="0.0" />
+      <xacro:property name="mono" value="false" />
+    </xacro:if>
+    <xacro:if value="${model == 'zedxonegs'}">
+      <xacro:property name="baseline" value="0.0" />
+      <xacro:property name="height" value="0.031" />
+      <xacro:property name="bottom_slope" value="0.0" />
+      <xacro:property name="screw_offset_x" value="0.0" />
+      <xacro:property name="screw_offset_z" value="-0.0155" />
+      <xacro:property name="optical_offset_x" value="0.0" />
+      <xacro:property name="mono" value="true" />
+    </xacro:if>
+    <xacro:if value="${model == 'zedxone4k'}">
+      <xacro:property name="baseline" value="0.0" />
+      <xacro:property name="height" value="0.031" />
+      <xacro:property name="bottom_slope" value="0.0" />
+      <xacro:property name="screw_offset_x" value="0.00" />
+      <xacro:property name="screw_offset_z" value="-0.0155" />
+      <xacro:property name="optical_offset_x" value="0.0" />
+      <xacro:property name="mono" value="true" />
     </xacro:if>
     <!-- Camera mounting point (the threaded screw hole in the bottom) -->
@@ -106,87 +131,104 @@
       <origin xyz="0 0 ${height/2}" rpy="0 ${bottom_slope} 0" />
     </joint>
-    <!-- Left Camera -->
-    <link name="${name}_left_camera_frame">
-      <xacro:if value="${model == 'virtual'}">
-        <visual>
-          <origin xyz="0 0 0" rpy="0 0 0"/>
-          <geometry>
-            <mesh filename="package://zed_interfaces/meshes/${model}.stl" />
-          </geometry>
-          <material name="${model}_mat" />
-        </visual>
-        <collision>
-          <origin xyz="0 0 0" rpy="0 0 0"/>
-          <geometry>
-            <mesh filename="package://zed_interfaces/meshes/${model}.stl" />
-          </geometry>
-        </collision>
+    <xacro:unless value="${mono}">
+      <!-- Left Camera -->
+      <link name="${name}_left_camera_frame">
+        <xacro:if value="${model == 'virtual'}">
+          <visual>
+            <origin xyz="0 0 0" rpy="0 0 0"/>
+            <geometry>
+              <mesh filename="package://zed_interfaces/meshes/${model}.stl" />
+            </geometry>
+            <material name="${model}_mat" />
+          </visual>
+          <collision>
+            <origin xyz="0 0 0" rpy="0 0 0"/>
+            <geometry>
+              <mesh filename="package://zed_interfaces/meshes/${model}.stl" />
+            </geometry>
+          </collision>
+        </xacro:if>
+      </link>
+      <joint name="${name}_left_camera_joint" type="fixed">
+        <parent link="${name}_camera_center"/>
+        <child link="${name}_left_camera_frame"/>
+        <origin xyz="${optical_offset_x} ${baseline/2} 0" rpy="0 0 0" />
+      </joint>
+      <link name="${name}_left_camera_optical_frame"/>
+      <joint name="${name}_left_camera_optical_joint" type="fixed">
+        <origin xyz="0 0 0" rpy="-${M_PI/2} 0.0 -${M_PI/2}"/>
+        <parent link="${name}_left_camera_frame"/>
+        <child link="${name}_left_camera_optical_frame"/>
+      </joint>
+      <!-- Right Camera -->
+      <link name="${name}_right_camera_frame">
+        <xacro:if value="${model == 'virtual'}">
+          <visual>
+            <origin xyz="0 0 0" rpy="0 0 0"/>
+            <geometry>
+              <mesh filename="package://zed_interfaces/meshes/${model}.stl" />
+            </geometry>
+            <material name="${model}_mat" />
+          </visual>
+          <collision>
+            <origin xyz="0 0 0" rpy="0 0 0"/>
+            <geometry>
+              <mesh filename="package://zed_interfaces/meshes/${model}.stl" />
+            </geometry>
+          </collision>
+        </xacro:if>
+      </link>
+      <joint name="${name}_right_camera_joint" type="fixed">
+        <parent link="${name}_camera_center"/>
+        <child link="${name}_right_camera_frame"/>
+        <origin xyz="${optical_offset_x} -${baseline/2} 0" rpy="0 0 0" />
+      </joint>
+      <link name="${name}_right_camera_optical_frame"/>
+      <joint name="${name}_right_camera_optical_joint" type="fixed">
+        <origin xyz="0 0 0" rpy="-${M_PI/2} 0.0 -${M_PI/2}"/>
+        <parent link="${name}_right_camera_frame"/>
+        <child link="${name}_right_camera_optical_frame"/>
+      </joint>
+      <!-- ZED2 Sensors -->
+      <xacro:if value="${model == 'zed2'}">
+        <link name="${name}_mag_link" />
+        <joint name="${name}_mag_joint" type="fixed">
+          <parent link="${name}_camera_center"/>
+          <child link="${name}_mag_link"/>
+          <origin xyz="0 0 0" rpy="0 0 0" />
+        </joint>
+        <link name="${name}_baro_link" />
+        <joint name="${name}_baro_joint" type="fixed">
+          <parent link="${name}_camera_center"/>
+          <child link="${name}_baro_link"/>
+          <origin xyz="0 0 0" rpy="0 0 0" />
+        </joint>
+        <link name="${name}_temp_left_link" />
+        <joint name="${name}_temp_left_joint" type="fixed">
+          <parent link="${name}_left_camera_frame"/>
+          <child link="${name}_temp_left_link"/>
+          <origin xyz="0 0 0" rpy="0 0 0" />
+        </joint>
+        <link name="${name}_temp_right_link" />
+        <joint name="${name}_temp_right_joint" type="fixed">
+          <parent link="${name}_right_camera_frame"/>
+          <child link="${name}_temp_right_link"/>
+          <origin xyz="0 0 0" rpy="0 0 0" />
+        </joint>
       </xacro:if>
-    </link>
-    <joint name="${name}_left_camera_joint" type="fixed">
-      <parent link="${name}_camera_center"/>
-      <child link="${name}_left_camera_frame"/>
-      <origin xyz="${optical_offset_x} ${baseline/2} 0" rpy="0 0 0" />
-    </joint>
-    <link name="${name}_left_camera_optical_frame"/>
-    <joint name="${name}_left_camera_optical_joint" type="fixed">
-      <origin xyz="0 0 0" rpy="-${M_PI/2} 0.0 -${M_PI/2}"/>
-      <parent link="${name}_left_camera_frame"/>
-      <child link="${name}_left_camera_optical_frame"/>
-    </joint>
-    <!-- Right Camera -->
-    <link name="${name}_right_camera_frame">
-      <xacro:if value="${model == 'virtual'}">
-        <visual>
-          <origin xyz="0 0 0" rpy="0 0 0"/>
-          <geometry>
-            <mesh filename="package://zed_interfaces/meshes/${model}.stl" />
-          </geometry>
-          <material name="${model}_mat" />
-        </visual>
-        <collision>
-          <origin xyz="0 0 0" rpy="0 0 0"/>
-          <geometry>
-            <mesh filename="package://zed_interfaces/meshes/${model}.stl" />
-          </geometry>
-        </collision>
-      </xacro:if>
-    </link>
-    <joint name="${name}_right_camera_joint" type="fixed">
-      <parent link="${name}_camera_center"/>
-      <child link="${name}_right_camera_frame"/>
-      <origin xyz="${optical_offset_x} -${baseline/2} 0" rpy="0 0 0" />
-    </joint>
-    <link name="${name}_right_camera_optical_frame"/>
-    <joint name="${name}_right_camera_optical_joint" type="fixed">
-      <origin xyz="0 0 0" rpy="-${M_PI/2} 0.0 -${M_PI/2}"/>
-      <parent link="${name}_right_camera_frame"/>
-      <child link="${name}_right_camera_optical_frame"/>
-    </joint>
-    <!-- ZED2 Sensors -->
-    <xacro:if value="${model == 'zed2'}">
-      <link name="${name}_mag_link" />
-      <joint name="${name}_mag_joint" type="fixed">
+    </xacro:unless>
+    <xacro:if value="${mono}">
+      <!-- Camera -->
+      <link name="${name}_camera_frame" />
+      <joint name="${name}_camera_joint" type="fixed">
         <parent link="${name}_camera_center"/>
-        <child link="${name}_mag_link"/>
-        <origin xyz="0 0 0" rpy="0 0 0" />
-      </joint>
-      <link name="${name}_baro_link" />
-      <joint name="${name}_baro_joint" type="fixed">
-        <parent link="${name}_camera_center"/>
-        <child link="${name}_baro_link"/>
-        <origin xyz="0 0 0" rpy="0 0 0" />
-      </joint>
-      <link name="${name}_temp_left_link" />
-      <joint name="${name}_temp_left_joint" type="fixed">
-        <parent link="${name}_left_camera_frame"/>
-        <child link="${name}_temp_left_link"/>
-        <origin xyz="0 0 0" rpy="0 0 0" />
-      </joint>
-      <link name="${name}_temp_right_link" />
-      <joint name="${name}_temp_right_joint" type="fixed">
-        <parent link="${name}_right_camera_frame"/>
-        <child link="${name}_temp_right_link"/>
-        <origin xyz="0 0 0" rpy="0 0 0" />
+        <child link="${name}_camera_frame"/>
+        <origin xyz="${optical_offset_x} 0 0" rpy="0 0 0" />
+      </joint>
+      <link name="${name}_camera_optical_frame"/>
+      <joint name="${name}_camera_optical_joint" type="fixed">
+        <origin xyz="0 0 0" rpy="-${M_PI/2} 0.0 -${M_PI/2}"/>
+        <parent link="${name}_camera_frame"/>
+        <child link="${name}_camera_optical_frame"/>
       </joint>
     </xacro:if>

Commit message: Add ZED X One HDR

File: zed_wrapper/urdf/include/materials.urdf.xacro (robot description, xacro)
@@ -43,3 +43,6 @@
         <color rgba="0.25 0.25 0.25 1.0"/>
     </material>
+    <material name="zedxonehdr_mat">
+        <color rgba="0.25 0.25 0.25 1.0"/>
+    </material>
 </robot>

File: zed_wrapper/urdf/zed_macro.urdf.xacro (robot description, xacro)
@@ -103,4 +103,13 @@
       <xacro:property name="screw_offset_x" value="0.00" />
       <xacro:property name="screw_offset_z" value="-0.0155" />
+      <xacro:property name="optical_offset_x" value="0.0" />
+      <xacro:property name="mono" value="true" />
+    </xacro:if>
+    <xacro:if value="${model == 'zedxonehdr'}">
+      <xacro:property name="baseline" value="0.0" />
+      <xacro:property name="height" value="0.025" />
+      <xacro:property name="bottom_slope" value="0.0" />
+      <xacro:property name="screw_offset_x" value="0.00" />
+      <xacro:property name="screw_offset_z" value="-0.0125" />
       <xacro:property name="optical_offset_x" value="0.0" />
       <xacro:property name="mono" value="true" />

Commit message: Add HDR cameras

File: zed_wrapper/urdf/include/materials.urdf.xacro (robot description, xacro)
@@ -34,4 +34,13 @@
         <color rgba="0.25 0.25 0.25 1.0"/>
     </material>
+    <material name="zedxhdr_mat">
+        <color rgba="0.25 0.25 0.25 1.0"/>
+    </material>
+    <material name="zedxhdrmini_mat">
+        <color rgba="0.25 0.25 0.25 1.0"/>
+    </material>
+    <material name="zedxhdrmax_mat">
+        <color rgba="0.25 0.25 0.25 1.0"/>
+    </material>
     <material name="virtual_mat">
         <color rgba="0.25 0.25 0.25 1.0"/>

File: zed_wrapper/urdf/zed_macro.urdf.xacro (robot description, xacro)
@@ -70,6 +70,33 @@
       <xacro:property name="mono" value="false" />
     </xacro:if>
+    <xacro:if value="${model == 'zedxhdr'}">
+      <xacro:property name="baseline" value="0.12" />
+      <xacro:property name="height" value="0.032" />
+      <xacro:property name="bottom_slope" value="0.0" />
+      <xacro:property name="screw_offset_x" value="0.0" />
+      <xacro:property name="screw_offset_z" value="-0.016" />
+      <xacro:property name="optical_offset_x" value="-0.01" />
+      <xacro:property name="mono" value="false" />
+    </xacro:if>
     <xacro:if value="${model == 'zedxm'}">
       <xacro:property name="baseline" value="0.05" />
+      <xacro:property name="height" value="0.032" />
+      <xacro:property name="bottom_slope" value="0.0" />
+      <xacro:property name="screw_offset_x" value="0.0" />
+      <xacro:property name="screw_offset_z" value="-0.016" />
+      <xacro:property name="optical_offset_x" value="-0.01" />
+      <xacro:property name="mono" value="false" />
+    </xacro:if>
+    <xacro:if value="${model == 'zedxhdrmini'}">
+      <xacro:property name="baseline" value="0.05" />
+      <xacro:property name="height" value="0.032" />
+      <xacro:property name="bottom_slope" value="0.0" />
+      <xacro:property name="screw_offset_x" value="0.0" />
+      <xacro:property name="screw_offset_z" value="-0.016" />
+      <xacro:property name="optical_offset_x" value="-0.01" />
+      <xacro:property name="mono" value="false" />
+    </xacro:if>
+    <xacro:if value="${model == 'zedxhdrmax'}">
+      <xacro:property name="baseline" value="0.170" />
       <xacro:property name="height" value="0.032" />
       <xacro:property name="bottom_slope" value="0.0" />
